File: electronics/ecu/connectors.kicad_sch (KiCad schematic)
At the start: 11 parts, among them J801 24V IN (+24V, 0V, PE), J802 CAN-FD1 engine W101 (H, L, GN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, J803 CAN-FD2 BOP W115, J804 CAN3 BMS W107, J805 RS-485 #1/#2 W105/W106 (A1, B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, J806 SPEED W102a/b (N1A+, N1A-, N1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, J807 SAFETY LOOP W103 (SMCU_PERMIT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, J808 DI 1-12 (24 V), J809 DI 13-24 (24 V), J810 RELAY RO1-6 (COM/NO), J811 RELAY RO7-12 (COM/NO)

Commit message: WIP: HVAC power modes, fire suppression, insulated-hall recheck; electrical EMS, boards, 3D room model; engine E1–E4 in progress
Co-Authored-By: Claude Fable 5.1 <noreply@anthropic.com>
Parts:
- J803: value CAN-FD2 BOP W115 -> CAN2 BMS W107
- J804: value CAN3 BMS W107 -> CAN3 spare
Changed lines of the file:
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@@
 			(effects (font (size 1.27 1.27)))
 		)
-		(property "Value" "CAN-FD2 BOP W115"
+		(property "Value" "CAN2 BMS W107"
 			(at 80.01 104.14 0)
 			(effects (font (size 1.27 1.27)))
@@
 			(effects (font (size 1.27 1.27)))
 		)
-		(property "Value" "CAN3 BMS W107"
+		(property "Value" "CAN3 spare"
 			(at 80.01 133.35 0)
 			(effects (font (size 1.27 1.27)))
